File: pcb/steno/steno-v2.kicad_pcb (KiCad board)
At the start: 2 copper layers, 195 x 70 mm, 59 parts, among them J1 Conn_01x02, J2 Conn_01x04, K1 KEYSW, K10 KEYSW, K11 KEYSW, K12 KEYSW, K13 KEYSW, K14 KEYSW, K15 KEYSW, K16 KEYSW, K17 KEYSW, K18 KEYSW, K19 KEYSW, K2 KEYSW, K20 KEYSW, K21 KEYSW, K22 KEYSW, K23 KEYSW, K24 KEYSW, K25 KEYSW, K26 KEYSW, K27 KEYSW, K28 KEYSW, K3 KEYSW, K4 KEYSW, K5 KEYSW, K6 KEYSW, K7 KEYSW, K8 KEYSW, K9 KEYSW, U1 Adafruit_Feather

Commit message: v2 KiCAD files
Parts:
- added D29: DIODE, Diode_THT:D_DO-34_SOD68_P7.62mm_Horizontal, B.Cu at (278.9, 71.3)
- added D30: DIODE, Diode_THT:D_DO-34_SOD68_P7.62mm_Horizontal, B.Cu at (282.6, 69.9)
- added J2: 503182-1852, misc:MOLEX_503182-1852, F.Cu at (233.3, 102.6)
- added K29: KEYSW, Keebio-Parts:Kailh-PG1350-1u-No-Clickhole, F.Cu at (345.4, 34.6)
- added K30: KEYSW, Keebio-Parts:Kailh-PG1350-1u-No-Clickhole, F.Cu at (351.3, 50.6)
- added R1: 10K, Resistor_SMD:R_0805_2012Metric, F.Cu at (230.6, 72.3)
- added U2: MT25QL128ABA1ESE, steno:SOIC-8, F.Cu at (231.6, 78.3)
- D1, D10, D11, D12, D13, D14, D15, D16, D17, D18, D19, D2, D20, D21, D22, D23, D24, D25, D26, D27, D28, D3, D4, D5, D6, D7, D8, D9: moved to B.Cu
- J1: moved to F.Cu
- moved K17 230.0 mm to (277.4, 58.3), turned to 200 degrees
- moved K18 212.0 mm to (292.3, 46.5), turned to 200 degrees
- moved K6 206.3 mm to (254.7, 48.5), turned to 200 degrees
- moved K19 195.7 mm to (311.3, 46.0), turned to 200 degrees
- moved K7 188.8 mm to (271.6, 42.3), turned to 200 degrees
- moved K20 180.4 mm to (334.3, 56.8), turned to 200 degrees
- moved K8 171.6 mm to (286.5, 30.5), turned to 200 degrees
- moved U1 164.7 mm to (233.1, 69.3), turned to 270 degrees
- moved D17 161.7 mm to (267.6, 75.4), turned to 290 degrees
- moved D18 158.1 mm to (273.2, 73.3), turned to 290 degrees
- moved K9 155.7 mm to (305.5, 30.0), turned to 200 degrees
- moved D19 152.6 mm to (277.0, 72.0), turned to 290 degrees
- moved D6 151.8 mm to (260.1, 78.1), turned to 290 degrees
- moved D20 151.2 mm to (284.5, 69.3), turned to 290 degrees
- moved D7 148.2 mm to (265.7, 76.1), turned to 290 degrees
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- renumbered J2 to J3
Connections:
- D10 pad 2: COL5 -> COL10
- D11 pad 2: COL6 -> COL1
- D12 pad 2: COL1 -> COL2
- D13 pad 2: COL2 -> COL3
- D14 pad 2: COL3 -> COL4
- D15 pad 2: COL4 -> COL5
- D16 pad 2: COL5 -> COL6
- D17 pad 2: COL1 -> COL7
- D18 pad 2: COL2 -> COL8
- D19 pad 2: COL3 -> COL9
- D20 pad 2: COL4 -> COL10
- D21 pad 2: COL5 -> COL1
- D22 pad 2: COL6 -> COL2
- D23 pad 2: COL1 -> COL3
- D24 pad 2: COL2 -> COL4
- D25 pad 2: COL3 -> COL5
- D26 pad 2: COL4 -> COL6
- D27 pad 2: COL5 -> COL7
- D28 pad 2: COL6 -> COL8
- D6 pad 2: COL1 -> COL6
- D7 pad 2: COL2 -> COL7
- D8 pad 2: COL3 -> COL8
- D9 pad 2: COL4 -> COL9
- K10 pad 1: ROW2 -> ROW1
- K12 pad 1: ROW3 -> ROW2
- K13 pad 1: ROW3 -> ROW2
- K14 pad 1: ROW3 -> ROW2
- K15 pad 1: ROW3 -> ROW2
- K16 pad 1: ROW3 -> ROW2
- K17 pad 1: ROW4 -> ROW2
- K18 pad 1: ROW4 -> ROW2
- K19 pad 1: ROW4 -> ROW2
- K20 pad 1: ROW4 -> ROW2
- K21 pad 1: ROW4 -> ROW3
- K22 pad 1: ROW4 -> ROW3
- K23 pad 1: ROW5 -> ROW3
- K24 pad 1: ROW5 -> ROW3
- K25 pad 1: ROW5 -> ROW3
- K26 pad 1: ROW5 -> ROW3
- K27 pad 1: ROW5 -> ROW3
- K28 pad 1: ROW5 -> ROW3
- K6 pad 1: ROW2 -> ROW1
- K7 pad 1: ROW2 -> ROW1
- K8 pad 1: ROW2 -> ROW1
- K9 pad 1: ROW2 -> ROW1
- U1 pad 2: Net-(U1-Pad2) -> COL5
- U1 pad 20: COL1 -> COL10
- U1 pad 21: COL2 -> COL9
- U1 pad 22: COL3 -> COL8
- U1 pad 23: COL4 -> COL7
- U1 pad 25: COL5 -> COL6
- U1 pad 26: COL6 -> CS
- U1 pad 3: Net-(U1-Pad3) -> COL4
- U1 pad 4: Net-(U1-Pad4) -> MISO
- U1 pad 5: Net-(U1-Pad5) -> MOSI
- U1 pad 6: Net-(U1-Pad6) -> SCLK
- U1 pad 7: Net-(U1-Pad7) -> COL3
- U1 pad 8: ROW5 -> COL2
- U1 pad 9: ROW4 -> COL1
Routing:
- net ROW4: track 231.7 -> 0.00 mm
- net GND: track 0.00 -> 193.5 mm, vias 0 -> 4
- net ROW3: track 193.6 -> 375.1 mm
- net ROW5: track 111.7 -> 0.00 mm
- net VCC: track 0.00 -> 107.5 mm
- net Net-(D29-Pad1): track 0.00 -> 91.7 mm
- net Net-(D30-Pad1): track 0.00 -> 79.8 mm
- net SCLK: track 0.00 -> 65.5 mm, vias 0 -> 1
- net BAT: track 0.00 -> 62.8 mm, vias 0 -> 1
- net MOSI: track 0.00 -> 61.8 mm, vias 0 -> 1
- net COL6: track 82.5 -> 23.2 mm
- net Net-(D11-Pad1): track 106.4 -> 50.0 mm
- net Net-(D5-Pad1): track 89.0 -> 35.2 mm
- net Net-(D16-Pad1): track 73.4 -> 19.8 mm
- net CS: track 0.00 -> 53.1 mm, vias 0 -> 1
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Other:
- board size 195 x 70 mm -> 258.9 x 93.1 mm

Commit message: Update PCB and footprints
Parts:
- removed J1: Conn_01x02, Connector_JST:JST_PH_B2B-PH-SM4-TB_1x02-1MP_P2.00mm_Vertical
- added BT1: Battery_Cell, Connector_JST:JST_PH_S2B-PH-SM4-TB_1x02-1MP_P2.00mm_Horizontal, F.Cu at (187.2, 120.5)
- U2: footprint steno:SOIC-8 -> Package_SO:SOP-8_5.28x5.23mm_P1.27mm
- moved K30 101.1 mm to (274.9, 116.8), turned to 180 degrees
- moved K20 98.0 mm to (256.9, 116.8), turned to 180 degrees
- moved K28 96.5 mm to (207.0, 132.6), turned to 180 degrees
- moved K29 96.1 mm to (274.9, 99.8), turned to 180 degrees
- moved K27 94.9 mm to (189.0, 132.6), turned to 180 degrees
- moved K26 93.6 mm to (171.0, 132.6), turned to 180 degrees
- moved K10 92.9 mm to (256.9, 99.8), turned to 180 degrees
- moved J2 90.0 mm to (146.3, 125.3), turned to 160 degrees
- moved K19 89.6 mm to (238.9, 98.8), turned to 180 degrees
- moved D18 87.9 mm to (192.1, 107.2), turned to 270 degrees
- moved D8 87.8 mm to (190.1, 107.2), turned to 270 degrees
- moved J3 87.6 mm to (128.4, 119.2), turned to 340 degrees
- moved D17 87.5 mm to (186.1, 107.2), turned to 270 degrees
- moved D7 87.3 mm to (184.1, 107.2), turned to 270 degrees
- moved D20 87.1 mm to (206.1, 107.2), turned to 270 degrees
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Connections:
- U1 pad 18: GND -> Net-(U1-Pad18)
Routing:
- net GND: track 193.5 -> 136.2 mm, vias 4 -> 3
- net Net-(D26-Pad1): track 19.5 -> 69.5 mm
- net ROW3: track 375.1 -> 393.1 mm
- net BAT: track 62.8 -> 48.0 mm, vias 1 -> 0
- net Net-(D27-Pad1): track 36.7 -> 48.1 mm
- net Net-(D7-Pad1): track 48.9 -> 39.0 mm
- net Net-(D8-Pad1): track 64.5 -> 56.8 mm
- net CS: track 53.1 -> 45.4 mm
- net Net-(D9-Pad1): track 69.6 -> 62.8 mm
- net COL8: track 39.0 -> 34.1 mm
- net COL9: track 46.1 -> 41.9 mm
- net COL7: track 31.8 -> 28.0 mm
- net Net-(D29-Pad1): track 91.7 -> 88.1 mm
- net Net-(D17-Pad1): track 30.8 -> 27.4 mm
- net MOSI: track 61.8 -> 58.7 mm, vias 1 -> 2
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Other:
- board size 258.9 x 93.1 mm -> 243.3 x 130.4 mm

Commit message: Update PCB
Parts:
- moved K30 41.6 mm to (282.0, 75.8), turned to 200 degrees
- moved K21 40.4 mm to (45.9, 75.8), turned to 160 degrees
- moved K29 40.0 mm to (276.2, 59.9), turned to 200 degrees
- moved K22 38.8 mm to (51.7, 59.8), turned to 160 degrees
- moved K20 35.8 mm to (265.1, 82.0), turned to 200 degrees
- moved K11 34.6 mm to (62.8, 82.0), turned to 160 degrees
- moved K10 33.9 mm to (259.3, 66.0), turned to 200 degrees
- moved K1 32.7 mm to (68.6, 66.0), turned to 160 degrees
- moved K19 27.8 mm to (242.1, 71.2), turned to 200 degrees
- moved K9 26.7 mm to (236.2, 55.2), turned to 200 degrees
- moved K12 26.6 mm to (85.9, 71.2), turned to 160 degrees
- moved K2 25.5 mm to (91.7, 55.2), turned to 160 degrees
- moved K28 25.1 mm to (223.7, 113.9), turned to 200 degrees
- moved K23 24.6 mm to (102.3, 113.9), turned to 160 degrees
- moved K27 21.8 mm to (206.7, 120.1), turned to 200 degrees
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Other:
- board size 243.3 x 130.4 mm -> 258.9 x 93.1 mm

Commit message: v3 component placement; Removed JST connector; Added OLED footprint
Parts:
- removed BT1: Battery_Cell, Connector_JST:JST_PH_S2B-PH-SM4-TB_1x02-1MP_P2.00mm_Horizontal
- removed J3: Conn_01x04, Connector_PinHeader_2.54mm:PinHeader_1x04_P2.54mm_Vertical
- removed the K10 at (259.3, 66.0)
- removed the K6 at (185.5, 73.7)
- removed the K7 at (202.4, 67.6)
- removed R1: 10K, Resistor_SMD:R_0805_2012Metric
- added J1: 503182-1852, misc:MOLEX_503182-1852, F.Cu at (161.7, 124.0)
- added K23: KEYSW, Keebio-Parts:Kailh-PG1350-1u-No-Clickhole, F.Cu at (196.5, 64.4)
- added K24: KEYSW, Keebio-Parts:Kailh-PG1350-1u-No-Clickhole, F.Cu at (179.4, 70.1)
- added K25: KEYSW, Keebio-Parts:Kailh-PG1350-1u-No-Clickhole, F.Cu at (275.9, 74.9)
- J2: value 503182-1852 -> Conn_01x04; footprint misc:MOLEX_503182-1852 -> steno:OLED
- moved K30 97.8 mm to (184.8, 86.2), turned to 198.4 degrees
- moved D21 86.4 mm to (198.5, 95.9), turned to 288.4 degrees
- moved K26 82.7 mm to (258.8, 80.6), turned to 198.4 degrees
- moved D7 78.3 mm to (115.3, 92.7), turned to 251.6 degrees
- moved D10 78.3 mm to (132.4, 98.4), turned to 251.6 degrees
- moved D8 78.1 mm to (121.0, 94.6), turned to 251.6 degrees
- moved K29 77.2 mm to (201.9, 80.5), turned to 198.4 degrees
- moved D9 76.2 mm to (128.6, 97.1), turned to 251.6 degrees
- moved D22 75.0 mm to (192.9, 97.8), turned to 288.4 degrees
- moved D25 68.6 mm to (206.1, 93.4), turned to 288.4 degrees
- moved K18 64.1 mm to (184.3, 122.8), turned to 198.4 degrees
- moved D23 59.9 mm to (187.2, 99.7), turned to 288.4 degrees
- moved K27 58.7 mm to (236.0, 69.2), turned to 198.4 degrees
- moved D24 50.5 mm to (183.4, 100.9), turned to 288.4 degrees
- moved D6 47.8 mm to (140.0, 100.9), turned to 251.6 degrees
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- renumbered K22 to K1, K13 to K10, K14 to K11, K15 to K12, K23 to K13, K24 to K14, K25 to K15, K1 to K2, K9 to K21, K8 to K22, K2 to K3, K3 to K4, K4 to K5, K5 to K6, K21 to K7, K11 to K8, K12 to K9
Connections:
- D10 pad 2: COL10 -> COL4
- D11 pad 2: COL1 -> COL5
- D12 pad 2: COL2 -> COL6
- D13 pad 2: COL3 -> COL1
- D14 pad 2: COL4 -> COL2
- D15 pad 2: COL5 -> COL3
- D16 pad 2: COL6 -> COL4
- D17 pad 2: COL7 -> COL5
- D18 pad 2: COL8 -> COL6
- D19 pad 2: COL9 -> COL1
- D20 pad 2: COL10 -> COL2
- D21 pad 2: COL1 -> COL3
- D22 pad 2: COL2 -> COL4
- D23 pad 2: COL3 -> COL5
- D24 pad 2: COL4 -> COL6
- D25 pad 2: COL5 -> COL1
- D26 pad 2: COL6 -> COL2
- D27 pad 2: COL7 -> COL3
- D28 pad 2: COL8 -> COL4
- D29 pad 2: COL9 -> COL5
- D30 pad 2: COL10 -> COL6
- D7 pad 2: COL7 -> COL1
- D8 pad 2: COL8 -> COL2
- D9 pad 2: COL9 -> COL3
- J2 pad 1: Net-(J2-Pad1) -> SDA
- J2 pad 2: CS -> SCL
- J2 pad 3: MOSI -> VCC
- J2 pad 4: VCC -> GND
- K1 pad 1: ROW3 -> ROW1
- K1 pad 2: Net-(D22-Pad1) -> Net-(D1-Pad1)
- K10 pad 2: Net-(D13-Pad1) -> Net-(D10-Pad1)
- K11 pad 2: Net-(D14-Pad1) -> Net-(D11-Pad1)
- K12 pad 2: Net-(D15-Pad1) -> Net-(D12-Pad1)
- K13 pad 2: Net-(D23-Pad1) -> Net-(D13-Pad1)
- K14 pad 2: Net-(D24-Pad1) -> Net-(D14-Pad1)
- K15 pad 2: Net-(D25-Pad1) -> Net-(D15-Pad1)
- K16 pad 1: ROW2 -> ROW3
- K17 pad 1: ROW2 -> ROW3
- K18 pad 1: ROW2 -> ROW3
- K19 pad 1: ROW2 -> ROW4
- K2 pad 2: Net-(D1-Pad1) -> Net-(D2-Pad1)
- K20 pad 1: ROW2 -> ROW4
- K21 pad 1: ROW1 -> ROW4
- K21 pad 2: Net-(D9-Pad1) -> Net-(D21-Pad1)
- K22 pad 1: ROW1 -> ROW4
- K22 pad 2: Net-(D8-Pad1) -> Net-(D22-Pad1)
- K26 pad 1: ROW3 -> ROW5
- K27 pad 1: ROW3 -> ROW5
- K28 pad 1: ROW3 -> ROW5
- K29 pad 1: ROW3 -> ROW5
- K3 pad 2: Net-(D2-Pad1) -> Net-(D3-Pad1)
- K30 pad 1: ROW3 -> ROW5
- K4 pad 2: Net-(D3-Pad1) -> Net-(D4-Pad1)
- K5 pad 2: Net-(D4-Pad1) -> Net-(D5-Pad1)
- K6 pad 2: Net-(D5-Pad1) -> Net-(D6-Pad1)
- K7 pad 1: ROW3 -> ROW2
- K7 pad 2: Net-(D21-Pad1) -> Net-(D7-Pad1)
- K8 pad 2: Net-(D11-Pad1) -> Net-(D8-Pad1)
- K9 pad 2: Net-(D12-Pad1) -> Net-(D9-Pad1)
- U1 pad 4: MISO -> MISO_DQ1
- U1 pad 5: MOSI -> MOSI_DQ0
- U2 pad 2: MISO -> MISO_DQ1
- U2 pad 3: Net-(R1-Pad1) -> DQ2
- U2 pad 5: MOSI -> MOSI_DQ0
- U2 pad 7: Net-(R1-Pad1) -> DQ3
Routing:
- net ROW3: track 393.1 -> 0.00 mm
- net ROW1: track 237.5 -> 0.00 mm
- net ROW2: track 232.8 -> 0.00 mm
- net GND: track 136.2 -> 0.00 mm, vias 3 -> 0
- net VCC: track 106.7 -> 0.00 mm
- net Net-(D29-Pad1): track 88.1 -> 0.00 mm
- net Net-(D22-Pad1): track 80.3 -> 0.00 mm
- net Net-(D30-Pad1): track 80.2 -> 0.00 mm
- net Net-(D26-Pad1): track 69.5 -> 0.00 mm
- net Net-(D10-Pad1): track 67.9 -> 0.00 mm
- net Net-(D21-Pad1): track 66.2 -> 0.00 mm
- net Net-(D2-Pad1): track 65.4 -> 0.00 mm
- net Net-(D9-Pad1): track 62.8 -> 0.00 mm
- net SCLK: track 62.5 -> 0.00 mm, vias 1 -> 0
- net MOSI: track 58.7 -> 0.00 mm, vias 2 -> 0
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Other:
- board size 258.9 x 93.1 mm -> 250.8 x 91.5 mm

Commit message: Routed and plotted v3
Parts:
- J1: value 503182-1852 -> Conn_01x02; footprint misc:MOLEX_503182-1852 -> Connector_PinHeader_2.54mm:PinHeader_1x02_P2.54mm_Vertical
- moved J1 40.4 mm to (155.5, 84.1), turned to 270 degrees
- moved J2 31.3 mm to (172.5, 113.1), turned to 180 degrees
- moved U2 14.2 mm to (154.0, 124.1), turned to 270 degrees
- moved D14 12.8 mm to (112.8, 91.7)
- moved D26 12.2 mm to (196.0, 91.0)
- moved D12 10.8 mm to (131.8, 98.0)
- moved D16 8.76 mm to (188.4, 93.6)
- moved D18 8.76 mm to (173.2, 98.6)
- moved D10 8.76 mm to (124.2, 95.5)
- moved K4 8.76 mm to (103.4, 50.1)
- moved U1 8.76 mm to (153.4, 105.1)
- moved K2 8.76 mm to (61.7, 61.5)
- moved D23 8.76 mm to (178.9, 96.7)
- moved D30 8.76 mm to (177.0, 97.4)
- moved K10 8.76 mm to (98.1, 66.2)
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Connections:
- J1 pad 1: Net-(J1-Pad1) -> BAT
- J1 pad 2: CS -> GND
- U1 pad 1: Net-(U1-Pad1) -> (no net)
- U1 pad 10: ROW3 -> COL3
- U1 pad 11: ROW2 -> COL2
- U1 pad 12: ROW1 -> COL1
- U1 pad 14: Net-(U1-Pad14) -> (no net)
- U1 pad 16: RST -> (no net)
- U1 pad 18: Net-(U1-Pad18) -> (no net)
- U1 pad 19: Net-(U1-Pad19) -> (no net)
- U1 pad 2: COL5 -> DQ3
- U1 pad 20: COL10 -> ROW1
- U1 pad 21: COL9 -> ROW2
- U1 pad 22: COL8 -> ROW4
- U1 pad 23: COL7 -> ROW5
- U1 pad 24: Net-(U1-Pad24) -> (no net)
- U1 pad 25: COL6 -> ROW3
- U1 pad 3: COL4 -> DQ2
- U1 pad 7: COL3 -> COL6
- U1 pad 8: COL2 -> COL5
- U1 pad 9: COL1 -> COL4
Routing:
- net ROW2: track 0.00 -> 160.7 mm, vias 0 -> 1
- net ROW1: track 0.00 -> 160.7 mm, vias 0 -> 1
- net ROW4: track 0.00 -> 156.3 mm, vias 0 -> 1
- net ROW5: track 0.00 -> 144.9 mm, vias 0 -> 1
- net ROW3: track 0.00 -> 135.1 mm
- net COL1: track 0.00 -> 105.3 mm
- net Net-(D19-Pad1): track 0.00 -> 94.2 mm
- net COL2: track 0.00 -> 93.2 mm
- net Net-(D1-Pad1): track 0.00 -> 83.1 mm
- net Net-(D25-Pad1): track 0.00 -> 82.1 mm
- net COL3: track 0.00 -> 80.9 mm
- net GND: track 0.00 -> 79.4 mm
- net VCC: track 0.00 -> 76.1 mm
- net Net-(D20-Pad1): track 0.00 -> 72.7 mm
- net Net-(D21-Pad1): track 0.00 -> 72.0 mm
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Other:
- board text added: "BAT"
- board text added: "GND"
