File: pcb/steno/mobile-steno.sch (KiCad schematic (older format))
At the start: 65 parts, among them J1 Conn_01x02, J2 Conn_01x04, J3 Conn_01x02, K1 KEYSW, K10 KEYSW, K11 KEYSW, K12 KEYSW, K13 KEYSW, K14 KEYSW, K15 KEYSW, K16 KEYSW, K17 KEYSW, K18 KEYSW, K19 KEYSW, K2 KEYSW, K20 KEYSW, K21 KEYSW, K22 KEYSW, K23 KEYSW, K24 KEYSW, K25 KEYSW, K26 KEYSW, K27 KEYSW, K28 KEYSW, K29 KEYSW, K3 KEYSW, K30 KEYSW, K4 KEYSW, K5 KEYSW, K6 KEYSW, K7 KEYSW, K8 KEYSW, K9 KEYSW, U1 Adafruit_Feather, U2 MT25QL128ABA1ESE

Commit message: Slightly improved layout and routing
- Moved thumb cluster to row 5 from 3
- Make row pins be in order
Connections:
- wire segments 119 -> 109
Changed lines of the file:
@@
 Text GLabel 7600 1550 0    50   Input ~ 0
 GND
-Text GLabel 8650 2450 2    50   BiDi ~ 0
+Text GLabel 8650 2150 2    50   BiDi ~ 0
 ROW3
 Text GLabel 7600 1950 0    50   BiDi ~ 0
@@
 $EndComp
 Wire Wire Line
-	5500 1300 6200 1300
-Wire Wire Line
-	6200 1400 6200 1300
-Wire Wire Line
 	6100 1700 6150 1700
 Wire Wire Line
@@
 $EndComp
 Wire Wire Line
-	5500 1850 6200 1850
-Wire Wire Line
-	6200 1950 6200 1850
-Wire Wire Line
 	6100 2250 6150 2250
 Wire Wire Line
@@
 $EndComp
 Wire Wire Line
-	5500 2400 6200 2400
-Wire Wire Line
-	6200 2500 6200 2400
-Wire Wire Line
 	6100 2800 6150 2800
 Connection ~ 6150 2250
-Connection ~ 5500 2400
-Connection ~ 5500 1850
-Connection ~ 5500 1300
 $Comp
 L canadian_parts:KEYSW K19
@@
 $EndComp
 Wire Wire Line
-	5500 2900 6200 2900
-Wire Wire Line
-	6200 3000 6200 2900
-Wire Wire Line
 	6100 3300 6150 3300
 Wire Wire Line
@@
 $EndComp
 Wire Wire Line
-	5500 3450 6200 3450
-Wire Wire Line
-	6200 3550 6200 3450
-Wire Wire Line
 	6100 3850 6150 3850
-Connection ~ 5500 3450
-Connection ~ 5500 2900
 Wire Wire Line
 	6150 3300 6150 2800
@@
 Text GLabel 6100 3850 3    50   BiDi ~ 0
 COL6
-Text GLabel 8650 2150 2    50   BiDi ~ 0
+Text GLabel 8650 2250 2    50   BiDi ~ 0
 ROW4
-Text GLabel 8650 2250 2    50   BiDi ~ 0
+Text GLabel 8650 2450 2    50   BiDi ~ 0
 ROW5
 Text GLabel 7600 2550 0    50   BiDi ~ 0
